Commit message: write desired control for 6 links, not 7. disable dummy end-effector link fully in urdf/m1n6s300.urdf remove the if simulator == "PyBullet": exception, deal with this inside kinova_pb.py add experimental/slow kinova_pb_pdcontrol.py (requires newer PyBullet with PD_CONTROL support in setJointMotorControlArray) remove precompiled binary Python files (pyc) they don't belong in git

File: Software/kinova_description/urdf/m1n6s300.urdf (robot description, URDF)
Before this commit: robot m1n6s300, 16 links, 15 joints
Links:
- removed link m1n6s300_end_effector
Joints:
- removed joint m1n6s300_joint_end_effector
